File: Kicad/Carte-mère/Carte-mère.kicad_pcb (KiCad board)
At the start: 2 copper layers, 26 parts, among them P1 CONN_01X08, P2 CONN_01X04, P3 CONN_01X06, P4 CONN_01X06, P5 CONN_01X04, P6 CONN_01X04, P7 CONN_01X02

Commit message: Mise à jour de la carte mère
Parts:
- added P10: CONN_01X04, Pin_Headers:Pin_Header_Straight_1x04, F.Cu at (181.6, 100.3)
- added P11: CONN_01X04, Pin_Headers:Pin_Header_Straight_1x04, F.Cu at (181.6, 104.1)
- added P8: CONN_01X04, Pin_Headers:Pin_Header_Straight_1x04, F.Cu at (144.8, 71.1)
- added P9: CONN_01X04, Pin_Headers:Pin_Header_Straight_1x04, F.Cu at (144.8, 67.3)
Routing:
- net +5V: track 283.2 -> 307.3 mm
- net Net-(ARD1-Pad1): track 47.9 -> 37.3 mm
- net Net-(ARD1-Pad29): track 79.1 -> 83.9 mm
- net Net-(ARD1-Pad28): track 53.9 -> 50.3 mm
- net +3.3V: track 141.5 -> 140.0 mm
- net Net-(ARD1-Pad11): track 84.5 -> 83.1 mm
- net Net-(ARD1-Pad8): track 57.5 -> 56.7 mm
Other:
- board text added: "+5V"
- board text added: "GND"
- board text added: "MOTEUR 1"
- board text added: "MOTEUR 2"

Commit message: Mise à jour du PCB
Parts:
- moved D1 15.3 mm to (157.5, 83.8), turned to 90 degrees
- moved R1 9.25 mm to (157.5, 87.6), turned to 90 degrees
Routing:
- net +5V: track 307.3 -> 220.5 mm, vias 0 -> 6
- net +BATT: track 115.2 -> 139.8 mm, vias 0 -> 2
- net Net-(ARD1-Pad17): track 65.5 -> 46.3 mm
- net GND: track 0.00 -> 17.6 mm, vias 0 -> 1
- net Net-(ARD1-Pad16): track 55.3 -> 41.2 mm
- net Net-(ARD1-Pad4): track 87.9 -> 74.4 mm, vias 0 -> 2
- net Net-(ARD1-Pad5): track 85.4 -> 75.1 mm, vias 0 -> 2
- net Net-(ARD1-Pad10): track 72.7 -> 82.2 mm
- net Net-(ARD1-Pad7): track 80.3 -> 89.7 mm, vias 0 -> 2
- net Net-(ARD1-Pad27): track 67.5 -> 60.4 mm, vias 0 -> 1
- net Net-(ARD1-Pad28): track 50.3 -> 56.6 mm
- net Net-(ARD1-Pad1): track 37.3 -> 41.8 mm
- net Net-(ARD1-Pad30): track 56.9 -> 60.8 mm
- net Net-(ARD1-Pad8): track 56.7 -> 59.9 mm, vias 0 -> 2
- net Net-(ARD1-Pad9): track 59.2 -> 61.9 mm
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
Commit message: Mise à jour du PCB
Routing:
- net (no net): track 362.2 -> 1.51 mm
Other:
- board outline added: 91.4 x 88.9 mm
Changed lines of the file:
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@@
     (links 80)
     (no_connects 0)
-    (area -118.237 63 197.492334 155.269001)
+    (area -118.237 63.424999 197.492334 155.269001)
     (thickness 1.6)
-    (drawings 9)
-    (tracks 330)
+    (drawings 13)
+    (tracks 326)
     (zones 0)
     (modules 30)
@@
     (0 F.Cu signal)
     (31 B.Cu signal)
-    (32 B.Adhes user)
-    (33 F.Adhes user)
-    (34 B.Paste user)
-    (35 F.Paste user)
-    (36 B.SilkS user)
-    (37 F.SilkS user)
-    (38 B.Mask user)
-    (39 F.Mask user)
-    (40 Dwgs.User user)
-    (41 Cmts.User user)
-    (42 Eco1.User user)
-    (43 Eco2.User user)
+    (32 B.Adhes user hide)
+    (33 F.Adhes user hide)
+    (34 B.Paste user hide)
+    (35 F.Paste user hide)
+    (36 B.SilkS user hide)
+    (37 F.SilkS user hide)
+    (38 B.Mask user hide)
+    (39 F.Mask user hide)
+    (40 Dwgs.User user hide)
+    (41 Cmts.User user hide)
+    (42 Eco1.User user hide)
+    (43 Eco2.User user hide)
     (44 Edge.Cuts user)
-    (45 Margin user)
-    (46 B.CrtYd user)
-    (47 F.CrtYd user)
-    (48 B.Fab user)
-    (49 F.Fab user)
+    (45 Margin user hide)
+    (46 B.CrtYd user hide)
+    (47 F.CrtYd user hide)
+    (48 B.Fab user hide)
+    (49 F.Fab user hide)
   )
   (setup
-    (last_trace_width 1)
+    (last_trace_width 0.254)
     (user_trace_width 0.5)
     (user_trace_width 1)
@@
     (visible_elements FFFFFF7F)
     (pcbplotparams
-      (layerselection 0x00030_80000001)
+      (layerselection 0x01000_80000001)
       (usegerberextensions false)
       (excludeedgelayer true)
@@
       (outputformat 1)
       (mirror false)
-      (drillshape 1)
+      (drillshape 0)
       (scaleselection 1)
-      (outputdirectory ""))
+      (outputdirectory Gerber/))
   )
   (net 0 "")
@@
     )
   )
+  (gr_line (start 104.775 152.4) (end 104.775 63.5) (angle 90) (layer Edge.Cuts) (width 0.15))
+  (gr_line (start 196.215 152.4) (end 104.775 152.4) (angle 90) (layer Edge.Cuts) (width 0.15))
+  (gr_line (start 196.215 63.5) (end 196.215 152.4) (angle 90) (layer Edge.Cuts) (width 0.15))
+  (gr_line (start 104.775 63.5) (end 196.215 63.5) (angle 90) (layer Edge.Cuts) (width 0.15))
   (gr_text "MOTEUR 2" (at 107.95 133.35 90) (layer F.SilkS)
     (effects (font (size 1.5 1.5) (thickness 0.3)))
@@
     (effects (font (size 1.5 1.5) (thickness 0.3)))
   )
-  (segment (start 104.775 63.5) (end 196.215 63.5) (width 1) (layer B.Cu) (net 0))
-  (segment (start 104.775 152.4) (end 104.775 63.5) (width 1) (layer B.Cu) (net 0))
-  (segment (start 196.215 152.4) (end 104.775 152.4) (width 1) (layer B.Cu) (net 0))
-  (segment (start 196.215 63.5) (end 196.215 152.4) (width 1) (layer B.Cu) (net 0))
   (segment (start -118.11 117.305) (end -117.94 117.475) (width 0.254) (layer F.Cu) (net 0))
   (segment (start -90.805 102.87) (end -90.17 102.87) (width 0.254) (layer B.Cu) (net 0))
@@
   (segment (start 132.715 109.22) (end 132.715 111.76) (width 1) (layer B.Cu) (net 11))
   (segment (start 132.715 134.62) (end 132.715 137.16) (width 1) (layer B.Cu) (net 11))
-  (segment (start 157.48 83.0707) (end 157.48 81.915) (width 0.5) (layer F.Cu) (net 12) (status 400000))
-  (segment (start 147.32 77.47) (end 147.32 76.2) (width 0.5) (layer B.Cu) (net 12) (status 800000))
+  (segment (start 157.48 83.0707) (end 157.48 81.915) (width 0.5) (layer F.Cu) (net 12))
+  (segment (start 147.32 77.47) (end 147.32 76.2) (width 0.5) (layer B.Cu) (net 12))
   (segment (start 146.685 78.105) (end 147.32 77.47) (width 0.5) (layer B.Cu) (net 12))
   (segment (start 146.685 81.28) (end 146.685 78.105) (width 0.5) (layer B.Cu) (net 12))
@@
   (segment (start 149.225 102.187006) (end 149.225 135.89) (width 1) (layer B.Cu) (net 22))
   (segment (start 154.94 96.472006) (end 149.225 102.187006) (width 1) (layer B.Cu) (net 22))
-  (segment (start 157.48 93.98) (end 157.48 91.44) (width 0.5) (layer B.Cu) (net 23) (status 400000))
-  (segment (start 157.48 91.44) (end 157.48 88.73) (width 0.5) (layer F.Cu) (net 23) (status 800000))
+  (segment (start 157.48 93.98) (end 157.48 91.44) (width 0.5) (layer B.Cu) (net 23))
+  (segment (start 157.48 91.44) (end 157.48 88.73) (width 0.5) (layer F.Cu) (net 23))
   (via (at 157.48 91.44) (size 0.889) (layers F.Cu B.Cu) (net 23))
   (segment (start 157.48 93.98) (end 157.48 96.52) (width 1) (layer B.Cu) (net 23))
@@
   (segment (start 140.97 148.59) (end 141.605 149.225) (width 1) (layer B.Cu) (net 25))
   (segment (start 140.97 146.685) (end 140.97 148.59) (width 1) (layer B.Cu) (net 25))
-  (segment (start 157.48 86.53) (end 157.48 84.5693) (width 0.5) (layer F.Cu) (net 26) (status C00000))
+  (segment (start 157.48 86.53) (end 157.48 84.5693) (width 0.5) (layer F.Cu) (net 26))
   (segment (start 111.76 129.54) (end 116.205 129.54) (width 1) (layer B.Cu) (net 27))
   (segment (start 118.745 134.62) (end 120.015 134.62) (width 1) (layer B.Cu) (net 27))
